Commit message: updated

File: wallbe/description/robot.urdf.xacro (robot description, xacro)
@@ -1,7 +1,8 @@
 <?xml version="1.0"?>
 <robot xmlns:xacro="http://www.ros.org/wiki/xacro"  name="robot">
-    <xacro:include filename="materials.xacro" />
-    <xacro:include filename="robot_core.xacro" />
-    <!-- <xacro:include filename="lidar.xacro" /> -->
+    <xacro:include filename="materials.urdf.xacro" />
+    <xacro:include filename="robot_core.urdf.xacro" />
+    <!-- <xacro:include filename="lidar.urdf.xacro" /> -->
+    <xacro:include filename="imu.urdf.xacro" />
     <xacro:include filename="ros2_control.xacro" />
 </robot>

File: wallbe/description/robot_core.urdf.xacro (robot description, xacro)
@@ -14,14 +14,22 @@
   <xacro:property name="caster_wheel_radius" value="0.015" />
   <xacro:property name="z_offset" value="-${base_height/2}" /> <!-- Space btw top of beam and the each joint -->
-  <!-- base_footprint Link -->
+  <!-- base_link -->
   <link name="base_footprint">
   </link>
-  <joint name="base_link_link" type="fixed">
-    <parent link="base_footprint"/>
-    <child link="base_link"/>
-    <origin xyz="0 0 0" rpy="0 0 0"/>
+  <!-- BASE_FOOTPRINT LINK -->
+  <joint name="base_footprint_joint" type="fixed">
+      <parent link="base_footprint"/>
+      <child link="base_link"/>
+      <origin xyz="0 0 0" rpy="0 0 0"/>
+  </joint>
+  <link name="base_link">
+  </link>
+  <joint name="chassis_joint" type="fixed">
+        <parent link="base_link"/>
+        <child link="chassis"/>
+        <origin xyz="0.09 0 0.02" rpy="0 0 0"/>
   </joint>
   <!-- Base Link -->
-  <link name="base_link">
+  <link name="chassis">
     <collision>
       <origin xyz="0.09 0 0.02" rpy="0 0 0"/>
