Commit message: fix slam_toolbox

File: wallbe/description/lidar.urdf.xacro (robot description, xacro)
@@ -9,7 +9,7 @@
     <link name="lidar_frame">
         <visual>
-            <origin xyz="0.0 0 0.1" rpy="${PI/2} 0 -${PI/2}"/>
+            <origin xyz="0.0 0 0.1" rpy="0 0 0"/>
             <geometry>
-                <mesh filename="package://wallBE/meshes/lidar.STL" scale="0.001 0.001 0.001"/>
+                <cylinder length="0.03" radius="0.02"/>
             </geometry>
             <material name="blue"/>

File: wallbe/description/robot.urdf.xacro (robot description, xacro)
@@ -1,8 +1,8 @@
 <?xml version="1.0"?>
 <robot xmlns:xacro="http://www.ros.org/wiki/xacro"  name="robot">
+    <xacro:include filename="ros2_control.xacro" />
     <xacro:include filename="materials.urdf.xacro" />
     <xacro:include filename="robot_core.urdf.xacro" />
-    <!-- <xacro:include filename="lidar.urdf.xacro" /> -->
+    <xacro:include filename="lidar.urdf.xacro" />
     <xacro:include filename="imu.urdf.xacro" />
-    <xacro:include filename="ros2_control.xacro" />
 </robot>

File: wallbe/description/robot_core.urdf.xacro (robot description, xacro)
@@ -14,22 +14,14 @@
   <xacro:property name="caster_wheel_radius" value="0.015" />
   <xacro:property name="z_offset" value="-${base_height/2}" /> <!-- Space btw top of beam and the each joint -->
-  <!-- base_link -->
+  <!-- base_footprint Link -->
   <link name="base_footprint">
   </link>
-  <!-- BASE_FOOTPRINT LINK -->
-  <joint name="base_footprint_joint" type="fixed">
-      <parent link="base_footprint"/>
-      <child link="base_link"/>
-      <origin xyz="0 0 0" rpy="0 0 0"/>
+  <joint name="base_link_link" type="fixed">
+    <parent link="base_footprint"/>
+    <child link="base_link"/>
+    <origin xyz="0 0 0" rpy="0 0 0"/>
   </joint>
+<!-- Base Link -->
   <link name="base_link">
-  </link>
-  <joint name="chassis_joint" type="fixed">
-        <parent link="base_link"/>
-        <child link="chassis"/>
-        <origin xyz="0.09 0 0.02" rpy="0 0 0"/>
-  </joint>
-  <!-- Base Link -->
-  <link name="chassis">
     <collision>
       <origin xyz="0.09 0 0.02" rpy="0 0 0"/>
@@ -46,135 +38,135 @@
     </visual>
   </link>
-    <joint name="left_wheel_joint" type="continuous">
-      <parent link="base_link"/>
-      <child link="left_wheel"/>
-      <origin xyz="0 -0.12 0" rpy="0 0 0"/>
-      <axis xyz="0 1 0"/>
-      <dynamics damping="0.2"/>
-    </joint>
-    <!-- left wheel Link -->
-    <link name="left_wheel">
-      <collision>
-        <origin xyz="0 0 0" rpy="${PI/2} 0 0"/>
-        <geometry>
-          <cylinder length="${wheel_len}" radius="${wheel_radius}"/>
-        </geometry>
-      </collision>
-      <visual>
-        <origin xyz="0 0 0" rpy="${PI/2} 0 0"/>
-        <geometry>
-          <cylinder length="${wheel_len}" radius="${wheel_radius}"/>
-        </geometry>
-        <material name="black"/>
-      </visual>
-    </link>
-    <joint name="right_wheel_joint" type="continuous">
-      <parent link="base_link"/>
-      <child link="right_wheel"/>
-      <origin xyz="0 0.12 0" rpy="0 0 0"/>
-      <axis xyz="0 1 0"/>
-      <dynamics damping="0.2"/>
-    </joint>
-    <!-- right wheel Link -->
-    <link name="right_wheel">
-      <collision>
-        <origin xyz="0 0 0" rpy="${PI/2} 0 0"/>
-        <geometry>
-          <cylinder length="${wheel_len}" radius="${wheel_radius}"/>
-        </geometry>
-      </collision>
-      <visual>
-        <origin xyz="0 0 0" rpy="${PI/2} 0 0"/>
-        <geometry>
-          <cylinder length="${wheel_len}" radius="${wheel_radius}"/>
-        </geometry>
-        <material name="black"/>
-      </visual>
-    </link>
-    <joint name="caster_frontal_wheel_joint" type="fixed">
-      <parent link="base_link"/>
-      <child link="caster_frontal_wheel"/>
-      <origin xyz="0.168 0 -0.015" rpy="0 0 0"/>
-    </joint>
-    <!-- caster frontal wheel Link -->
-    <link name="caster_frontal_wheel">
-      <collision>
-        <origin xyz="0 0 0" rpy="0 0 0"/>
-        <geometry>
-          <sphere radius="${caster_wheel_radius}"/>
-        </geometry>
-      </collision>
-      <visual>
-        <origin xyz="0 0 0" rpy="0 0 0"/>
-        <geometry>
-          <sphere radius="${caster_wheel_radius}"/>
-        </geometry>
-        <material name="white"/>
-      </visual>
-    </link>
-    <joint name="hub_joint" type="fixed">
-      <parent link="base_link"/>
-      <child link="hub"/>
-      <origin xyz="0.168 0 0.005" rpy="0 0 0"/>
-    </joint>
-<!-- Hub Link -->
-    <link name="hub">
-      <collision>
-        <origin xyz="0 0 0" rpy="0 0 0"/>
-        <geometry>
-          <box size="0.05 0.046 0.03"/>
-        </geometry>
-      </collision>
-      <visual>
-        <origin xyz="0 0 0" rpy="0 0 0"/>
-        <geometry>
-          <box size="0.05 0.046 0.03"/>
-        </geometry>
-        <material name="blue"/>
-      </visual>
-    </link>
-    <joint name="left_motor_joint" type="fixed">
-      <parent link="base_link"/>
-      <child link="left_motor"/>
-      <origin xyz="0 -0.0725 0" rpy="0 0 0"/>
-      <axis xyz="0 1 0"/>
-    </joint>
-    <!-- left motor Link -->
-    <link name="left_motor">
-      <collision>
-        <origin xyz="0 0 0" rpy="${PI/2} 0 0"/>
-        <geometry>
-          <cylinder length="0.08" radius="0.0125"/>
-        </geometry>
-      </collision>
-      <visual>
-        <origin xyz="0 0 0" rpy="${PI/2} 0 0"/>
-        <geometry>
-          <cylinder length="0.08" radius="0.0125"/>
-        </geometry>
-        <material name="green"/>
-      </visual>
-    </link>
-    <joint name="right_motor_joint" type="fixed">
-      <parent link="base_link"/>
-      <child link="right_motor"/>
-      <origin xyz="0 0.0725 0" rpy="0 0 0"/>
-      <axis xyz="0 1 0"/>
-    </joint>
-    <!-- right motor Link -->
-    <link name="right_motor">
-      <collision>
-        <origin xyz="0 0 0" rpy="${PI/2} 0 0"/>
-        <geometry>
-          <cylinder length="0.08" radius="0.0125"/>
-        </geometry>
-      </collision>
-      <visual>
-        <origin xyz="0 0 0" rpy="${PI/2} 0 0"/>
-        <geometry>
-          <cylinder length="0.08" radius="0.0125"/>
-        </geometry>
-        <material name="green"/>
-      </visual>
-    </link>
+  <joint name="left_wheel_joint" type="continuous">
+    <parent link="base_link"/>
+    <child link="left_wheel"/>
+    <origin xyz="0 -0.12 0" rpy="0 0 0"/>
+    <axis xyz="0 1 0"/>
+    <dynamics damping="0.2"/>
+  </joint>
+  <!-- left wheel Link -->
+  <link name="left_wheel">
+    <collision>
+      <origin xyz="0 0 0" rpy="${PI/2} 0 0"/>
+      <geometry>
+        <cylinder length="${wheel_len}" radius="${wheel_radius}"/>
+      </geometry>
+    </collision>
+    <visual>
+      <origin xyz="0 0 0" rpy="${PI/2} 0 0"/>
+      <geometry>
+        <cylinder length="${wheel_len}" radius="${wheel_radius}"/>
+      </geometry>
+      <material name="black"/>
+    </visual>
+  </link>
+  <joint name="right_wheel_joint" type="continuous">
+    <parent link="base_link"/>
+    <child link="right_wheel"/>
+    <origin xyz="0 0.12 0" rpy="0 0 0"/>
+    <axis xyz="0 1 0"/>
+    <dynamics damping="0.2"/>
+  </joint>
+  <!-- right wheel Link -->
+  <link name="right_wheel">
+    <collision>
+      <origin xyz="0 0 0" rpy="${PI/2} 0 0"/>
+      <geometry>
+        <cylinder length="${wheel_len}" radius="${wheel_radius}"/>
+      </geometry>
+    </collision>
+    <visual>
+      <origin xyz="0 0 0" rpy="${PI/2} 0 0"/>
+      <geometry>
+        <cylinder length="${wheel_len}" radius="${wheel_radius}"/>
+      </geometry>
+      <material name="black"/>
+    </visual>
+  </link>
+  <joint name="caster_frontal_wheel_joint" type="fixed">
+    <parent link="base_link"/>
+    <child link="caster_frontal_wheel"/>
+    <origin xyz="0.168 0 -0.015" rpy="0 0 0"/>
+  </joint>
+  <!-- caster frontal wheel Link -->
+  <link name="caster_frontal_wheel">
+    <collision>
+      <origin xyz="0 0 0" rpy="0 0 0"/>
+      <geometry>
+        <sphere radius="${caster_wheel_radius}"/>
+      </geometry>
+    </collision>
+    <visual>
+      <origin xyz="0 0 0" rpy="0 0 0"/>
+      <geometry>
+        <sphere radius="${caster_wheel_radius}"/>
+      </geometry>
+      <material name="white"/>
+    </visual>
+  </link>
+  <joint name="hub_joint" type="fixed">
+    <parent link="base_link"/>
+    <child link="hub"/>
+    <origin xyz="0.168 0 0.005" rpy="0 0 0"/>
+  </joint>
+  <!-- Hub Link -->
+  <link name="hub">
+    <collision>
+      <origin xyz="0 0 0" rpy="0 0 0"/>
+      <geometry>
+        <box size="0.05 0.046 0.03"/>
+      </geometry>
+    </collision>
+    <visual>
+      <origin xyz="0 0 0" rpy="0 0 0"/>
+      <geometry>
+        <box size="0.05 0.046 0.03"/>
+      </geometry>
+      <material name="blue"/>
+    </visual>
+  </link>
+  <joint name="left_motor_joint" type="fixed">
+    <parent link="base_link"/>
+    <child link="left_motor"/>
+    <origin xyz="0 -0.0725 0" rpy="0 0 0"/>
+    <axis xyz="0 1 0"/>
+  </joint>
+  <!-- left motor Link -->
+  <link name="left_motor">
+    <collision>
+      <origin xyz="0 0 0" rpy="${PI/2} 0 0"/>
+      <geometry>
+        <cylinder length="0.08" radius="0.0125"/>
+      </geometry>
+    </collision>
+    <visual>
+      <origin xyz="0 0 0" rpy="${PI/2} 0 0"/>
+      <geometry>
+        <cylinder length="0.08" radius="0.0125"/>
+      </geometry>
+      <material name="green"/>
+    </visual>
+  </link>
+  <joint name="right_motor_joint" type="fixed">
+    <parent link="base_link"/>
+    <child link="right_motor"/>
+    <origin xyz="0 0.0725 0" rpy="0 0 0"/>
+    <axis xyz="0 1 0"/>
+  </joint>
+  <!-- right motor Link -->
+  <link name="right_motor">
+    <collision>
+      <origin xyz="0 0 0" rpy="${PI/2} 0 0"/>
+      <geometry>
+        <cylinder length="0.08" radius="0.0125"/>
+      </geometry>
+    </collision>
+    <visual>
+      <origin xyz="0 0 0" rpy="${PI/2} 0 0"/>
+      <geometry>
+        <cylinder length="0.08" radius="0.0125"/>
+      </geometry>
+      <material name="green"/>
+    </visual>
+  </link>
 </robot>
